Commit message: Support for MoveIt and Gazebo

File: src/mycobot_280pi/mycobot_280pi_description/urdf/control/gazebo_sim_ros2_control.urdf.xacro (robot description, xacro)
@@ -5,5 +5,5 @@
             <gazebo>
                 <plugin filename="gz_ros2_control-system" name="gz_ros2_control::GazeboSimROS2ControlPlugin">
-                    <parameters>$(find mycobot_moveit_config)/config/${robot_name}/ros2_controllers.yaml</parameters>
+                    <parameters>$(find mycobot_280pi_moveit2_config)/config/${robot_name}/ros2_controllers.yaml</parameters>
                     <ros>
                         <remapping>/controller_manager/robot_description:=/robot_description</remapping>

File: src/mycobot_280pi/mycobot_280pi_description/urdf/robots/mycobot_280pi.urdf.xacro (robot description, xacro)
@@ -1,5 +1,5 @@
 <?xml version="1.0"?>
-<robot xmlns:xacro="http://www.ros.org/wiki/xacro" name="mycobot_280">
-    <xacro:arg name="robot_name" default="mycobot_280"/>
+<robot xmlns:xacro="http://www.ros.org/wiki/xacro" name="mycobot_280pi">
+    <xacro:arg name="robot_name" default="mycobot_280pi"/>
     <xacro:arg name="add_world" default="true"/>
     <xacro:arg name="base_link" default="link1"/>

File: src/mycobot_280pi/mycobot_280pi_description/urdf/sensors/intel_rgbd_cam_d435.urdf.xacro (robot description, xacro)
@@ -64,5 +64,5 @@
         <origin xyz="0 0 0" rpy="${M_PI/2} 0.0 ${M_PI/2}"/>
         <geometry>
-          <mesh filename="file://$(find mycobot_description)/meshes/d435/visual/d435.stl" />
+          <mesh filename="file://$(find mycobot_280pi_description)/meshes/d435/visual/d435.stl" />
         </geometry>
         <material name="aluminum">
