Commit message: Corrected initial gripper poition

File: src/mycobot_280pi/mycobot_280pi_description/urdf/robots/mycobot_280pi.urdf.xacro (robot description, xacro)
@@ -40,5 +40,5 @@
                 parent="$(arg flange_link)"
                 prefix="$(arg prefix)">
-                <origin xyz="0 0 0.034" rpy="1.579 0 0"/>
+                <origin xyz="0 0 0.034" rpy="1.579 0 0.785398"/>
             </xacro:adaptive_gripper>
         </xacro:if>
